File: modules/as3310-adsr/pcb/front/as3310-adsr_front.kicad_pcb (KiCad board)
At the start: 2 copper layers, 18.3 x 107.4 mm, 22 parts, among them J1 Pin Header 1x9, J2 Thonkiconn SM, J3 Thonkiconn SM

Commit message: modules: as3310-adsr: front: upgrade to kicad 6
Connections:
- J2 pad TN: (no net) -> unconnected-(J2-PadTN)
- J3 pad TN: (no net) -> unconnected-(J3-PadTN)
Other:
- net class Default removed
