File: modules/midi-splitter/pcb/back/midi-splitter_back.kicad_pcb (KiCad board)
At the start: 2 copper layers, 17.8 x 68.2 mm, 10 parts, among them J1 Pin Socket 1x7, J2 IDC Header 2x8, U1 74HC14

Commit message: modules: midi-splitter: back: upgrade to kicad 6
Connections:
- J2 pad 1: (no net) -> unconnected-(J2-Pad1)
- J2 pad 10: (no net) -> unconnected-(J2-Pad10)
- J2 pad 13: (no net) -> unconnected-(J2-Pad13)
- J2 pad 14: (no net) -> unconnected-(J2-Pad14)
- J2 pad 15: (no net) -> unconnected-(J2-Pad15)
- J2 pad 16: (no net) -> unconnected-(J2-Pad16)
- J2 pad 2: (no net) -> unconnected-(J2-Pad2)
- J2 pad 9: (no net) -> unconnected-(J2-Pad9)
Other:
- net class Default removed
