File: modules/midi-splitter/pcb/front/midi-splitter_front.kicad_pcb (KiCad board)
At the start: 2 copper layers, 17.8 x 98.7 mm, 23 parts, among them J1 Pin Header 1x7, J2 Thonkiconn ST, J3 Thonkiconn ST, J4 Thonkiconn ST, J5 Thonkiconn ST, U1 6N137

Commit message: modules: midi-splitter: front: upgrade to kicad 6
Connections:
- J2 pad S: (no net) -> unconnected-(J2-PadS)
- U1 pad 1: (no net) -> unconnected-(U1-Pad1)
- U1 pad 7: (no net) -> unconnected-(U1-Pad7)
Other:
- net class Default removed
