File: prototype-pcbs/4hp/4hp.kicad_pcb (KiCad board)
At the start: 2 copper layers, 17.8 x 109.2 mm, 289 parts

Commit message: prototype-pcbs: 4hp: upgrade to kicad 6
Other:
- net class Default removed
