File: prototype-pcbs/8hp/8hp.kicad_pcb (KiCad board)
At the start: 2 copper layers, 38.1 x 109.2 mm, 633 parts

Commit message: prototype-pcbs: 8hp: upgrade to kicad 6
Other:
- net class Default removed
