File: prototype-pcbs/12hp/12hp.kicad_pcb (KiCad board)
At the start: 2 copper layers, 58.4 x 109.2 mm, 977 parts

Commit message: prototype-pcbs: 12hp: upgrade to kicad 6
Other:
- net class Default removed
