File: modules/midi-oscillator/pcb/back/midi-oscillator_back.kicad_sch (KiCad schematic)
At the start: 17 parts, among them J1 JST XH 1x5, J2 IDC Header 2x8, J3 Pin Socket 1x14, U1 Raspberry Pi Pico, U2 MCP4822, U3 MCP4822, U4 24LC512

Commit message: modules: midi-oscillator: back: new revision 1.1
Parts:
- U2, U3, U4: footprint Package_DIP:DIP-8_W7.62mm_LongPads -> Package_DIP:DIP-8_W7.62mm
Connections:
- net +3V3 renamed +3.3V
Changed lines of the file:
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@@
   (title_block
     (title "midi-oscillator back")
-    (date "2021-12-15")
-    (rev "1.0")
+    (date "2022-07-08")
+    (rev "1.1")
     (comment 3 "Released under CERN Open Hardware Licence Version 2 - Strongly Reciprocal")
     (comment 4 "Designed by: Rafael G. Martins")
@@
     (property "Reference" "U3" (id 0) (at 137.16 98.2726 0))
     (property "Value" "MCP4822" (id 1) (at 137.16 100.584 0))
-    (property "Footprint" "Package_DIP:DIP-8_W7.62mm_LongPads" (id 2) (at 157.48 120.65 0)
+    (property "Footprint" "Package_DIP:DIP-8_W7.62mm" (id 2) (at 157.48 120.65 0)
       (effects (font (size 1.27 1.27)) hide)
     )
@@
     (property "Reference" "U2" (id 0) (at 137.16 55.0926 0))
     (property "Value" "MCP4822" (id 1) (at 137.16 57.404 0))
-    (property "Footprint" "Package_DIP:DIP-8_W7.62mm_LongPads" (id 2) (at 157.48 77.47 0)
+    (property "Footprint" "Package_DIP:DIP-8_W7.62mm" (id 2) (at 157.48 77.47 0)
       (effects (font (size 1.27 1.27)) hide)
     )
@@
     (property "Reference" "U4" (id 0) (at 184.15 57.6326 0))
     (property "Value" "24LC512" (id 1) (at 184.15 59.944 0))
-    (property "Footprint" "Package_DIP:DIP-8_W7.62mm_LongPads" (id 2) (at 184.15 69.85 0)
+    (property "Footprint" "Package_DIP:DIP-8_W7.62mm" (id 2) (at 184.15 69.85 0)
       (effects (font (size 1.27 1.27)) hide)
     )
@@
     )
     (path "/00000000-0000-0000-0000-000061e3ff8a"
-      (reference "U2") (unit 1) (value "MCP4822") (footprint "Package_DIP:DIP-8_W7.62mm_LongPads")
+      (reference "U2") (unit 1) (value "MCP4822") (footprint "Package_DIP:DIP-8_W7.62mm")
     )
     (path "/00000000-0000-0000-0000-000061bd15e6"
-      (reference "U3") (unit 1) (value "MCP4822") (footprint "Package_DIP:DIP-8_W7.62mm_LongPads")
+      (reference "U3") (unit 1) (value "MCP4822") (footprint "Package_DIP:DIP-8_W7.62mm")
     )
     (path "/00000000-0000-0000-0000-000061e3ffc6"
-      (reference "U4") (unit 1) (value "24LC512") (footprint "Package_DIP:DIP-8_W7.62mm_LongPads")
-    )
-  )
+      (reference "U4") (unit 1) (value "24LC512") (footprint "Package_DIP:DIP-8_W7.62mm")
+    )
+  )
